File: smartled_controll.kicad_pcb (KiCad board)
At the start: 2 copper layers, 61.2 x 43.7 mm, 89 parts, among them J1 Conn_01x04, SW1 SW_Push, U1 OC5028B, U2 MAX485E, U3 PY32F003F1xUx, U4 OC5864, U5 need chooice, U6 OC5028B, U7 need chooice, U8 OC5028B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

Commit message: 添加GND,VINP等覆铜（提交前已清除填充来减小文件大小，请在KiCAD重新填充）
Routing:
- net /PWM1: track 28.6 -> 29.6 mm
- added copper zone on F.Cu, net /VIN+
- added copper zone on F.Cu, net /VIN-
- added copper zone on B.Cu, net GND
- added copper zone on F.Cu, net GND
- added copper zone on F.Cu, net VINP
Changed lines of the file:
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@@
+	)
+	(segment
+		(start 142.28 66.86)
+		(end 145.77 70.35)
+		(width 0.25)
+		(layer "B.Cu")
+		(net 6)
 	)
 	(segment
@@
 	)
 	(segment
+		(start 136.185 66.86)
+		(end 142.28 66.86)
+		(width 0.25)
+		(layer "B.Cu")
+		(net 6)
+	)
+	(segment
 		(start 149.245 78.435)
 		(end 154.21 78.435)
@@
 	)
 	(segment
-		(start 139.675 70.35)
-		(end 145.77 70.35)
-		(width 0.25)
-		(layer "B.Cu")
-		(net 6)
-	)
-	(segment
 		(start 155.545 66.885)
 		(end 152.77325 66.885)
@@
 		(start 145.77 70.35)
 		(end 145.77 74.96)
-		(width 0.25)
-		(layer "B.Cu")
-		(net 6)
-	)
-	(segment
-		(start 136.185 66.86)
-		(end 139.675 70.35)
 		(width 0.25)
 		(layer "B.Cu")
@@
 	)
 	(segment
-		(start 145.145 72.77)
-		(end 145.48825 72.77)
-		(width 0.25)
-		(layer "F.Cu")
-		(net 38)
-	)
-	(segment
 		(start 137.81 89.9)
 		(end 138.15 90.24)
@@
 		(net 38)
 	)
+	(segment
+		(start 143.56835 71.5)
+		(end 144.83835 72.77)
+		(width 0.25)
+		(layer "F.Cu")
+		(net 38)
+	)
+	(segment
+		(start 144.83835 72.77)
+		(end 145.48825 72.77)
+		(width 0.25)
+		(layer "F.Cu")
+		(net 38)
+	)
+	(segment
+		(start 142.16 71.5)
+		(end 143.56835 71.5)
+		(width 0.25)
+		(layer "F.Cu")
+		(net 38)
+	)
 	(via
-		(at 145.145 72.77)
+		(at 142.16 71.5)
 		(size 0.6)
 		(drill 0.3)
@@
 	)
 	(segment
+		(start 140.89 72.77)
+		(end 137.61 72.77)
+		(width 0.2)
+		(layer "B.Cu")
+		(net 38)
+	)
+	(segment
 		(start 134.22 86.31)
+		(end 137.81 89.9)
+		(width 0.2)
+		(layer "B.Cu")
+		(net 38)
+	)
+	(segment
+		(start 142.16 71.5)
+		(end 140.89 72.77)
+		(width 0.2)
+		(layer "B.Cu")
+		(net 38)
+	)
+	(segment
+		(start 134.22 76.16)
+		(end 134.22 86.31)
+		(width 0.2)
+		(layer "B.Cu")
+		(net 38)
+	)
+	(segment
+		(start 137.61 72.77)
 		(end 134.22 76.16)
-		(width 0.2)
-		(layer "B.Cu")
-		(net 38)
-	)
-	(segment
-		(start 137.61 72.77)
-		(end 145.145 72.77)
-		(width 0.2)
-		(layer "B.Cu")
-		(net 38)
-	)
-	(segment
-		(start 137.81 89.9)
-		(end 134.22 86.31)
-		(width 0.2)
-		(layer "B.Cu")
-		(net 38)
-	)
-	(segment
-		(start 134.22 76.16)
-		(end 137.61 72.77)
 		(width 0.2)
 		(layer "B.Cu")
@@
 		(net 61)
 	)
+	(zone
+		(net 25)
+		(net_name "/VIN-")
+		(layer "F.Cu")
+		(hatch edge 0.5)
+		(priority 3)
+		(connect_pads yes
+			(clearance 0.5)
+		)
+		(min_thickness 0.25)
+		(filled_areas_thickness no)
+		(fill
+			(thermal_gap 0.5)
+			(thermal_bridge_width 0.5)
+			(smoothing fillet)
+			(radius 0.5)
+		)
+		(polygon
+			(pts
+				(xy 187.2 76.89) (xy 187.2 75.3) (xy 189.2 75.29) (xy 190.65 76.67) (xy 191.75 76.68) (xy 192.54 77.52)
+				(xy 191.79 78.36) (xy 188.63 78.34)
+			)
+		)
+	)
+	(zone
+		(net 23)
+		(net_name "/VIN+")
+		(layer "F.Cu")
+		(hatch edge 0.5)
+		(priority 2)
+		(connect_pads yes
+			(clearance 0.5)
+		)
+		(min_thickness 0.25)
+		(filled_areas_thickness no)
+		(fill
+			(thermal_gap 0.5)
+			(thermal_bridge_width 0.5)
+			(smoothing fillet)
+			(radius 0.5)
+		)
+		(polygon
+			(pts
+				(xy 184.78 72.36) (xy 184.79 70.62) (xy 189.11 70.66) (xy 192.59 74.13) (xy 192.59 75.82) (xy 190.9 75.82)
+				(xy 189.185 74.1) (xy 187.47 72.38)
+			)
+		)
+	)
+	(zone
+		(net 7)
+		(net_name "VINP")
+		(layer "F.Cu")
+		(hatch edge 0.5)
+		(priority 1)
+		(connect_pads yes
+			(clearance 0.5)
+		)
+		(min_thickness 0.25)
+		(filled_areas_thickness no)
+		(fill
+			(thermal_gap 0.5)
+			(thermal_bridge_width 0.5)
+			(smoothing fillet)
+			(radius 0.5)
+		)
+		(polygon
+			(pts
+				(xy 167.47 59.17) (xy 164.83 63.37) (xy 164.92 68.88) (xy 155.97 68.99) (xy 151.72 64.49) (xy 151.77 59.42)
+				(xy 148.11 59.41) (xy 146.135 62.685) (xy 135.78 73.18) (xy 135.77 76.57) (xy 138.53 76.58) (xy 140.76 74.34)
+				(xy 140.77 71.69) (xy 145.4 67.04) (xy 150.42 67.02) (xy 155.81 72.61) (xy 162.15 73.5) (xy 166.66 73.58)
+				(xy 179.15 73.59) (xy 179.15 69.95) (xy 180.64 69.49) (xy 185.59 64.92) (xy 188.51 64.53) (xy 190.57 59.42)
+				(xy 187.12 59.38) (xy 183.045 63.51) (xy 178.97 67.64) (xy 170.94 67.58) (xy 170.94 59.15)
+			)
+		)
+	)
+	(zone
+		(net 5)
+		(net_name "GND")
+		(layers "F.Cu" "B.Cu")
+		(hatch edge 0.5)
+		(connect_pads yes
+			(clearance 0.5)
+		)
+		(min_thickness 0.25)
+		(filled_areas_thickness no)
+		(fill
+			(thermal_gap 0.5)
+			(thermal_bridge_width 0.5)
+			(smoothing fillet)
+			(radius 0.5)
+		)
+		(polygon
+			(pts
+				(xy 132.4 52) (xy 193.6 52) (xy 193.6 95.7) (xy 132.4 95.7)
+			)
+		)
+	)
 	(group "电源输入电路"
