File: 4channels/smartled_controll.kicad_pcb (KiCad board)
At the start: 2 copper layers, 61.2 x 43.7 mm, 100 parts, among them J1 Conn_01x04, J2 Conn_01x02, SW1 SW_Push, U1 OC5028B, U2 MAX485E, U3 PY32F003F1xUx, U4 OC5864, U5 SGM2033-3.3, U6 OC5028B, U7 GS8521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

Commit message: MAX485 RO添加稳压二极管做电平转换
Parts:
- added D16: 2.0V, Diode_SMD:D_SOD-523, F.Cu at (143.2, 89.2)
Connections:
- U2 pad 1: /MAX485_RO -> Net-(D16-K)
Routing:
- net /MAX485_RO: track 7.27 -> 2.14 mm
- net Net-(D16-K): track 0.00 -> 3.89 mm
