File: 4channels/smartled_controll.kicad_sch (KiCad schematic)
At the start: 103 parts, among them J1 Conn_01x04, J2 Conn_01x02, SW1 SW_Push, U1 OC5028B, U2 MAX485E, U3 PY32F003F1xUx, U4 OC5864, U5 SGM2033-3.3, U6 OC5028B, U7 GS8521, U8 OC5028B, U9 OC5028B, Y1 Crystal_GND23

Commit message: 按照OC5028B数据手册，散热焊接与SW引脚连接 修复Out-与In-短路问题，已有PCB在散热焊盘涂阻焊油处理
Parts:
- U1, U6, U8, U9: footprint Package_SO:HSOP-8-1EP_3.9x4.9mm_P1.27mm_EP2.41x3.1mm_ThermalVias -> project_footprints:HSOP-8-1EP_3.9x4.9mm_P1.27mm_EP2.41x3.1mm_ThermalVias_0.3_0.6mm
Connections:
- net GND: no longer U1.9 (GND), U6.9 (GND), U8.9 (GND), U9.9 (GND)
- net at D9.2 (A), L4.1, U6.4 (SW): now also U6.9 (EP)
- net at D10.2 (A), L5.1, U8.4 (SW): now also U8.9 (EP)
- net at D5.2 (A), L3.1, U1.4 (SW): now also U1.9 (EP)
- net at D11.2 (A), L6.1, U9.4 (SW): now also U9.9 (EP)
Changed lines of the file:
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@@
 			)
 		)
-		(property "Footprint" "Package_SO:HSOP-8-1EP_3.9x4.9mm_P1.27mm_EP2.41x3.1mm_ThermalVias"
+		(property "Footprint" "project_footprints:HSOP-8-1EP_3.9x4.9mm_P1.27mm_EP2.41x3.1mm_ThermalVias_0.3_0.6mm"
 			(at 80.01 180.34 0)
 			(effects
@@
 			)
 		)
-		(property "Footprint" "Package_SO:HSOP-8-1EP_3.9x4.9mm_P1.27mm_EP2.41x3.1mm_ThermalVias"
+		(property "Footprint" "project_footprints:HSOP-8-1EP_3.9x4.9mm_P1.27mm_EP2.41x3.1mm_ThermalVias_0.3_0.6mm"
 			(at 80.01 142.24 0)
 			(effects
@@
 			)
 		)
-		(property "Footprint" "Package_SO:HSOP-8-1EP_3.9x4.9mm_P1.27mm_EP2.41x3.1mm_ThermalVias"
+		(property "Footprint" "project_footprints:HSOP-8-1EP_3.9x4.9mm_P1.27mm_EP2.41x3.1mm_ThermalVias_0.3_0.6mm"
 			(at 38.1 142.24 0)
 			(effects
@@
 			)
 		)
-		(property "Footprint" "Package_SO:HSOP-8-1EP_3.9x4.9mm_P1.27mm_EP2.41x3.1mm_ThermalVias"
+		(property "Footprint" "project_footprints:HSOP-8-1EP_3.9x4.9mm_P1.27mm_EP2.41x3.1mm_ThermalVias_0.3_0.6mm"
 			(at 34.29 180.34 0)
 			(effects
