File: smartled_2channels/smartled_2channels.kicad_sch (KiCad schematic)
At the start: 97 parts, among them Q1 Q_NMOS_GSD, SW1 SW_Push, U1 OC5028B, U2 MAX485E, U3 PY32F003F1xUx, U4 OC5864, U5 SGM2033-3.3, U6 OC5028B, U7 GS8521

Commit message: 按照OC5028B数据手册，散热焊接与SW引脚连接 修复Out-与In-短路问题，已有PCB在散热焊盘涂阻焊油处理
Connections:
- net GND: no longer U1.9 (GND), U6.9 (GND)
- net at D9.2 (A), L4.1, U6.4 (SW): now also U6.9 (EP)
- net at D5.2 (A), L3.1, U1.4 (SW): now also U1.9 (EP)
